File: Hardware/Connections.sch (KiCad schematic (older format))
At the start: 22 parts, among them J1 USB, P1 DisplayTop1, P10 Reservoir, P11 JTAG, P2 DisplayTop2, P3 DisplayBottom1, P4 DisplayBottom2, P5 Rotary, P6 FuncBtn, P7 REED, P8 CONN_2, P9 I2C

Commit message: Created PCB for new version with parallel display & sram
Parts:
- removed P1: DisplayTop1, symbol CONN_8
- removed P2: DisplayTop2, symbol CONN_8
- removed P3: DisplayBottom1, symbol CONN_8
- removed P4: DisplayBottom2, symbol CONN_8
- added C20: 470nF, SM1812, symbol C
- added R14: 10k, symbol R
- added U3: Display, symbol CONN_17X2
- added U6: LM3940, symbol LM3940
- P4: renamed from P8; value CONN_2 -> Flowmeter
- renumbered P6 to P2, P7 to P3, P9 to P5, P10 to P6, P11 to P7, P5 to P8, R9 to R10, R10 to R7, R7 to R8, R8 to R9
Connections:
- net labels removed: USART1_RX, USART1_TX
- wire segments 85 -> 95
Other:
- moved on the sheet: P2, P3, P4, P6, P7, P8, R10, R11, R12, R13, R4, R5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

Commit message: added 5V net and some text to the pcb
Parts:
- added D2, D3: 3.6V, symbol ZENER
- added P9: Voltmeter, symbol CONN_2
- added R16: 16V-20V, varistor-R-5, symbol VARISTOR-5
- added R17: 7,5, symbol R
- added R18: 1,5, symbol R
Connections:
- net labels added: +5V, Voltmeter
- wire segments 95 -> 112
Other:
- note added: "0 - 16V, max. 20V"
- note added: "0-3.3V"
- note added: "Voltmeter Connector"
- moved on the sheet: P7, R11, R12, R13
