File: Hardware/mainboard.sch (KiCad schematic (older format))
At the start: 24 parts, among them U1 STM32F10XZX, X1 32.768, X2 8MHz

Commit message: Created PCB for new version with parallel display & sram
Parts:
- added P1: VCC, symbol CONN_2
Connections:
- net labels added: A1, A10, A11, A12, A13, A14, A15, A16, A17, A2, A3, A4, A5, A6, A7, A8, A9, FLOW, NBL0, NBL1, OSC32_IN, OSC32_OUT, OSC_IN, OSC_OUT, RES, SLED, VBAT
- net labels removed: USART1_RX, USART1_TX
Other:
- note removed: "Todo: SDCARD, VCC Pins"

Commit message: added 5V net and some text to the pcb
Parts:
- added P10: VCC-5V, symbol CONN_2
Connections:
- net labels added: +5V, VOLTMETER
- wire segments 128 -> 131
Other:
- moved on the sheet: P1
