File: Hardware/sensors/gimmicks.sch (KiCad schematic (older format))
At the start: 3 parts, among them P601 BMP085, P602 ArduIMU, P603 HMC6352

Commit message: sensor board first version
Parts:
- added P604: ArduIMU2, symbol CONN_5
Connections:
- net +3.3V: now also P604.5
- net GND: now also P604.4
- new net GYRO_OUT2: P604.3
- new net GYRO_PD2: P604.2
- new net GYRO_ST2: P604.1
Changed lines of the file:
@@
-EESchema Schematic File Version 2  date Do 10 Mär 2011 16:21:43 CET
+EESchema Schematic File Version 2  date Do 17 Mär 2011 20:34:15 CET
 LIBS:power
 LIBS:device
@@
 Sheet 6 8
 Title ""
-Date "10 mar 2011"
+Date "17 mar 2011"
 Rev ""
 Comp ""
@@
 Comment4 ""
 $EndDescr
+$Comp
+L CONN_5 P604
+U 1 1 4D7BAFA5
+P 2450 2400
+F 0 "P604" V 2400 2400 50  0000 C CNN
+F 1 "ArduIMU2" V 2500 2400 50  0000 C CNN
+	1    2450 2400
+	-1   0    0    1
+$EndComp
+$Comp
+L +3.3V #PWR046
+U 1 1 4D7BAFA4
+P 2850 2200
+F 0 "#PWR046" H 2850 2160 30  0001 C CNN
+F 1 "+3.3V" H 2850 2310 30  0000 C CNN
+	1    2850 2200
+	1    0    0    -1
+$EndComp
+$Comp
+L GND #PWR047
+U 1 1 4D7BAFA3
+P 2850 2300
+F 0 "#PWR047" H 2850 2300 30  0001 C CNN
+F 1 "GND" H 2850 2230 30  0001 C CNN
+	1    2850 2300
+	0    -1   -1   0
+$EndComp
+Text HLabel 3000 2400 2    60   Output ~ 0
+GYRO_OUT2
+Text Notes 3550 2400 0    60   ~ 0
+(Analog)
+Text HLabel 3000 2500 2    60   Input ~ 0
+GYRO_PD2
+Text HLabel 3000 2600 2    60   Input ~ 0
+GYRO_ST2
+Wire Wire Line
+	2850 2500 3000 2500
+Wire Wire Line
+	2850 2400 3000 2400
+Wire Wire Line
+	3000 2600 2850 2600
 Wire Wire Line
 	1250 3350 1050 3350
@@
 	1050 3250 1250 3250
 $Comp
-L GND #PWR038
+L GND #PWR048
 U 1 1 4D74DE0C
 P 1050 3550
-F 0 "#PWR038" H 1050 3550 30  0001 C CNN
+F 0 "#PWR048" H 1050 3550 30  0001 C CNN
 F 1 "GND" H 1050 3480 30  0001 C CNN
 	1    1050 3550
@@
 $EndComp
 $Comp
-L +3.3V #PWR039
+L +3.3V #PWR049
 U 1 1 4D74DE09
 P 1050 3450
-F 0 "#PWR039" H 1050 3410 30  0001 C CNN
+F 0 "#PWR049" H 1050 3410 30  0001 C CNN
 F 1 "+3.3V" H 1050 3560 30  0000 C CNN
 	1    1050 3450
@@
 GYRO_OUT
 $Comp
-L GND #PWR040
+L GND #PWR050
 U 1 1 4D74DC76
 P 1100 2300
-F 0 "#PWR040" H 1100 2300 30  0001 C CNN
+F 0 "#PWR050" H 1100 2300 30  0001 C CNN
 F 1 "GND" H 1100 2230 30  0001 C CNN
 	1    1100 2300
@@
 $EndComp
 $Comp
-L +3.3V #PWR041
+L +3.3V #PWR051
 U 1 1 4D74DC72
 P 1100 2200
-F 0 "#PWR041" H 1100 2160 30  0001 C CNN
+F 0 "#PWR051" H 1100 2160 30  0001 C CNN
 F 1 "+3.3V" H 1100 2310 30  0000 C CNN
 	1    1100 2200
@@
 Gyro:\nhttp://www.watterott.com/de/ArduIMU-Sensor-Board-Six-Degrees-of-Freedom-Daughter
 $Comp
-L +3.3V #PWR042
+L +3.3V #PWR052
 U 1 1 4D74DB69
 P 1050 1500
-F 0 "#PWR042" H 1050 1460 30  0001 C CNN
+F 0 "#PWR052" H 1050 1460 30  0001 C CNN
 F 1 "+3.3V" H 1050 1610 30  0000 C CNN
 	1    1050 1500
@@
 $EndComp
 $Comp
-L GND #PWR043
+L GND #PWR053
 U 1 1 4D74DB62
 P 1050 1400
-F 0 "#PWR043" H 1050 1400 30  0001 C CNN
+F 0 "#PWR053" H 1050 1400 30  0001 C CNN
 F 1 "GND" H 1050 1330 30  0001 C CNN
 	1    1050 1400
