File: Hardware/sensors/power.sch (KiCad schematic (older format))
At the start: 11 parts, among them P501 MainPwr, U501 LM317

Commit message: changes to mcu, new format and using a display adapter board
Changed lines of the file:
@@
-EESchema Schematic File Version 2  date Mi 18 Mai 2011 15:58:13 CEST
+EESchema Schematic File Version 2  date Mi 18 Mai 2011 21:50:26 CEST
 LIBS:power
 LIBS:device
@@
 Comment4 ""
 $EndDescr
-$Comp
-L GND #PWR041
+Connection ~ 2300 3700
+Wire Wire Line
+	2300 3600 2300 3700
+Connection ~ 2000 2550
+Wire Wire Line
+	2000 2450 2000 2550
+Wire Wire Line
+	3150 1800 3300 1800
+Connection ~ 3300 1900
+Wire Wire Line
+	3450 1900 2500 1900
+Wire Wire Line
+	1350 2550 1350 2100
+Connection ~ 2500 3700
+Wire Wire Line
+	2850 3700 2200 3700
+Connection ~ 2850 3300
+Wire Wire Line
+	4300 1050 4650 1050
+Wire Wire Line
+	5050 1650 5200 1650
+Connection ~ 2700 1900
+Wire Wire Line
+	1350 1900 2000 1900
+Wire Wire Line
+	3000 1900 3000 1950
+Wire Wire Line
+	3300 1800 3300 1900
+Connection ~ 3000 1900
+Wire Wire Line
+	5750 1050 5750 1650
+Wire Wire Line
+	5750 1650 5700 1650
+Connection ~ 5750 1050
+Wire Wire Line
+	5050 1750 5050 1550
+Connection ~ 5050 1650
+Wire Wire Line
+	1450 3300 1600 3300
+Connection ~ 2500 3300
+Wire Wire Line
+	1350 2100 1500 2100
+Wire Wire Line
+	1950 2550 2050 2550
+Wire Wire Line
+	2700 1900 2700 1950
+Wire Wire Line
+	3350 3300 2200 3300
+Connection ~ 3150 3300
+Wire Wire Line
+	6150 1050 5450 1050
+Connection ~ 5900 1050
+$Comp
+L PWR_FLAG #FLG2
+U 1 1 4DD422F8
+P 2300 3600
+F 0 "#FLG2" H 2300 3870 30  0001 C CNN
+F 1 "PWR_FLAG" H 2300 3830 30  0000 C CNN
+	1    2300 3600
+	1    0    0    -1
+$EndComp
+$Comp
+L PWR_FLAG #FLG5
+U 1 1 4DD422ED
+P 6150 1050
+F 0 "#FLG5" H 6150 1320 30  0001 C CNN
+F 1 "PWR_FLAG" H 6150 1280 30  0000 C CNN
+	1    6150 1050
+	1    0    0    -1
+$EndComp
+$Comp
+L PWR_FLAG #FLG1
+U 1 1 4DD422E6
+P 2000 2450
+F 0 "#FLG1" H 2000 2720 30  0001 C CNN
+F 1 "PWR_FLAG" H 2000 2680 30  0000 C CNN
+	1    2000 2450
+	1    0    0    -1
+$EndComp
+$Comp
+L PWR_FLAG #FLG4
+U 1 1 4DD422DF
+P 3350 3300
+F 0 "#FLG4" H 3350 3570 30  0001 C CNN
+F 1 "PWR_FLAG" H 3350 3530 30  0000 C CNN
+	1    3350 3300
+	1    0    0    -1
+$EndComp
+$Comp
+L PWR_FLAG #FLG3
+U 1 1 4DD422D4
+P 3150 1800
+F 0 "#FLG3" H 3150 2070 30  0001 C CNN
+F 1 "PWR_FLAG" H 3150 2030 30  0000 C CNN
+	1    3150 1800
+	1    0    0    -1
+$EndComp
+$Comp
+L GND #PWR46
 U 1 1 4D782864
 P 2700 2350
-F 0 "#PWR041" H 2700 2350 30  0001 C CNN
+F 0 "#PWR46" H 2700 2350 30  0001 C CNN
 F 1 "GND" H 2700 2280 30  0001 C CNN
 	1    2700 2350
 	1    0    0    -1
 $EndComp
-Wire Wire Line
-	2700 1900 2700 1950
-Wire Wire Line
-	1950 2550 2050 2550
-Wire Wire Line
-	1500 2100 1350 2100
-Connection ~ 2500 3300
-Wire Wire Line
-	1450 3300 1600 3300
-Connection ~ 5050 1650
-Wire Wire Line
-	5050 1750 5050 1550
-Connection ~ 5750 1050
-Wire Wire Line
-	5700 1650 5750 1650
-Wire Wire Line
-	5750 1650 5750 1050
-Connection ~ 3000 1900
-Wire Wire Line
-	3300 1900 3300 1800
-Wire Wire Line
-	3000 1900 3000 1950
-Wire Wire Line
-	1350 1900 2000 1900
-Connection ~ 2700 1900
-Wire Wire Line
-	5450 1050 5900 1050
-Wire Wire Line
-	5050 1650 5200 1650
-Wire Wire Line
-	4300 1050 4650 1050
-Wire Wire Line
-	3150 3300 2200 3300
-Connection ~ 2850 3300
-Wire Wire Line
-	2850 3700 2200 3700
-Connection ~ 2500 3700
-Wire Wire Line
-	1350 2100 1350 2550
-Wire Wire Line
-	3450 1900 2500 1900
-Connection ~ 3300 1900
 $Comp
 L ZENER D501
@@
 EXTVCC
 $Comp
-L GNDA #PWR042
+L GNDA #PWR44
 U 1 1 4D74EFD7
 P 2050 2550
-F 0 "#PWR042" H 2050 2550 40  0001 C CNN
+F 0 "#PWR44" H 2050 2550 40  0001 C CNN
 F 1 "GNDA" H 2050 2480 40  0000 C CNN
 	1    2050 2550
@@
 $EndComp
 $Comp
-L GND #PWR043
+L GND #PWR45
 U 1 1 4D74EDED
 P 2200 3700
-F 0 "#PWR043" H 2200 3700 30  0001 C CNN
+F 0 "#PWR45" H 2200 3700 30  0001 C CNN
 F 1 "GND" H 2200 3630 30  0001 C CNN
 	1    2200 3700
@@
 $EndComp
 $Comp
-L VAA #PWR49
+L VAA #PWR48
 U 1 1 4D74EDD2
 P 3150 3300
-F 0 "#PWR49" H 3150 3360 30  0001 C CNN
+F 0 "#PWR48" H 3150 3360 30  0001 C CNN
 F 1 "VAA" H 3150 3410 30  0000 C CNN
 	1    3150 3300
@@
 $EndComp
 $Comp
-L +3.3V #PWR044
+L +3.3V #PWR42
 U 1 1 4D74ED3E
 P 1450 3300
-F 0 "#PWR044" H 1450 3260 30  0001 C CNN
+F 0 "#PWR42" H 1450 3260 30  0001 C CNN
 F 1 "+3.3V" H 1450 3410 30  0000 C CNN
 	1    1450 3300
@@
 $EndComp
 $Comp
-L GND #PWR045
+L GND #PWR51
 U 1 1 4D744126
 P 5050 2250
-F 0 "#PWR045" H 5050 2250 30  0001 C CNN
+F 0 "#PWR51" H 5050 2250 30  0001 C CNN
 F 1 "GND" H 5050 2180 30  0001 C CNN
 	1    5050 2250
@@
 $EndComp
 $Comp
-L +3.3V #PWR046
+L +3.3V #PWR52
 U 1 1 4D7440F5
 P 5900 1050
-F 0 "#PWR046" H 5900 1010 30  0001 C CNN
+F 0 "#PWR52" H 5900 1010 30  0001 C CNN
 F 1 "+3.3V" H 5900 1160 30  0000 C CNN
 	1    5900 1050
@@
 $EndComp
 $Comp
-L +12V #PWR047
+L +12V #PWR50
 U 1 1 4D7440F1
 P 4300 1050
-F 0 "#PWR047" H 4300 1000 20  0001 C CNN
+F 0 "#PWR50" H 4300 1000 20  0001 C CNN
 F 1 "+12V" H 4300 1150 30  0000 C CNN
 	1    4300 1050
@@
 $EndComp
 $Comp
-L +12V #PWR048
+L +12V #PWR49
 U 1 1 4D743E7E
 P 3300 1800
-F 0 "#PWR048" H 3300 1750 20  0001 C CNN
+F 0 "#PWR49" H 3300 1750 20  0001 C CNN
 F 1 "+12V" H 3300 1900 30  0000 C CNN
 	1    3300 1800
@@
 $EndComp
 $Comp
-L GND #PWR049
+L GND #PWR47
 U 1 1 4D743E56
 P 3000 2350
-F 0 "#PWR049" H 3000 2350 30  0001 C CNN
+F 0 "#PWR47" H 3000 2350 30  0001 C CNN
 F 1 "GND" H 3000 2280 30  0001 C CNN
 	1    3000 2350
@@
 $EndComp
 $Comp
-L GND #PWR050
+L GND #PWR43
 U 1 1 4D743D88
 P 1500 2100
-F 0 "#PWR050" H 1500 2100 30  0001 C CNN
+F 0 "#PWR43" H 1500 2100 30  0001 C CNN
 F 1 "GND" H 1500 2030 30  0001 C CNN
 	1    1500 2100
