File: Hardware/sensors/sensors.sch (KiCad schematic (older format))
At the start: 34 parts, among them P701 Sensors, U701 BAS40-04, U702 BAS40-04, U703 BAS40-04, U704 BAS40-04, U705 BAS40-04, U706 BAS40-04, U707 BAS40-04, U708 DS18B20, U709 DS18B20

Commit message: sensor board first version
Parts:
- removed P701: Sensors, symbol CONN_8
- added C708: 100nF, symbol C
- added P701: sens1, symbol CONN_2
- added P702: sens2, symbol CONN_2
- added P703: sens3, symbol CONN_2
- added P704: sens4, symbol CONN_2
- added R718: 2k7, symbol R
- added R719: 10k, symbol R
- added U710: BAS40-04, symbol BAS40-04
- U708, U709: value DS18B20 -> DS1820
Connections:
- net labels added: SupplyVoltage
- wire segments 68 -> 93
